File: 260929_KiCadPractice_Nichika.kicad_pcb (KiCad board)
At the start: 2 copper layers, 120 x 90 mm, 31 parts, among them J1 Micro_SD_Card_Det_Hirose_DM3AT, J2 Conn_01x02_Socket, U1 Qwiic-SAM-M8Q, U2 AE_BME280, U3 E22-900T30D_E220-900T22S(JP)_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, U4 NJM7805FA-ND

Commit message: feat(pcb): New PCB Design is created.
Parts:
- moved R2 230.4 mm to (53.5, 73.3)
- moved R3 229.8 mm to (53.4, 70.8)
- moved C8 200.4 mm to (94.7, 107.6), turned to 90 degrees
- moved D1 199.9 mm to (120.3, 42.7)
- moved C3 196.2 mm to (81.1, 47.3), turned to 90 degrees
- moved R4 194.9 mm to (87.5, 63.9), turned to 90 degrees
- moved R5 192.8 mm to (89.4, 63.9), turned to 90 degrees
- moved R1 191.5 mm to (114.3, 130.8)
- moved R7 191.0 mm to (97.0, 63.9), turned to 90 degrees
- moved R6 190.7 mm to (91.3, 63.9), turned to 90 degrees
- moved S1 190.6 mm to (133.3, 55.1), turned to 90 degrees
- moved J2 189.3 mm to (135.8, 45.2), turned to 180 degrees
- moved R8 188.8 mm to (98.9, 63.9), turned to 90 degrees
- moved U2 187.6 mm to (116.3, 69.8)
- moved U3 186.9 mm to (70.3, 113.8), turned to -90 degrees
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Routing:
- net +3.3V: track 23.6 -> 268.4 mm, vias 0 -> 12
- net +5V: track 0.00 -> 198.0 mm, vias 0 -> 3
- net /LoRa_TXD: track 0.00 -> 119.7 mm, vias 0 -> 2
- net /LoRa_AUX: track 0.00 -> 112.1 mm, vias 0 -> 2
- net /LoRa_M0: track 0.00 -> 108.7 mm, vias 0 -> 1
- net /LoRa_RXD: track 0.00 -> 105.6 mm, vias 0 -> 1
- net /LoRa_M1: track 0.00 -> 97.0 mm, vias 0 -> 1
- net /GNSS_TXD: track 0.00 -> 87.0 mm, vias 0 -> 3
- net /GNSS_RXD: track 0.00 -> 86.2 mm, vias 0 -> 3
- net /I2C1_SDA: track 0.00 -> 60.3 mm, vias 0 -> 1
- net /SPI0_RX: track 0.00 -> 60.2 mm, vias 0 -> 2
- net /I2C1_SCL: track 0.00 -> 60.2 mm, vias 0 -> 1
- net /SPI0_SCK: track 0.00 -> 41.9 mm, vias 0 -> 1
- net /SPI0_CS: track 0.00 -> 39.1 mm, vias 0 -> 1
- net /SPI0_TX: track 0.00 -> 33.1 mm, vias 0 -> 1
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- removed copper zone on B.Cu, net GND
- removed copper zone on F.Cu, net GND
Other:
- board size 120 x 90 mm -> 100 x 100 mm

Commit message: fix(pcb): Board fixed.
Parts:
- moved D1 5.18 mm to (125.5, 42.6), turned to 180 degrees
Routing:
- net Net-(D1-K): track 0.00 -> 10.5 mm
- net +7.5V: track 9.53 -> 12.8 mm
- net +5V: track 198.0 -> 201.2 mm
- net GND: vias 0 -> 352
- net /LoRa_AUX: vias 2 -> 3
- added copper zone on B.Cu, net GND
- added copper zone on F.Cu, net GND

Commit message: feat(pcb): Silkscreen updated.
Routing:
- net /LoRa_AUX: vias 3 -> 2
Other:
- board text added: "+"
- board text added: "-"
- board text added: "Anode"
- board text added: "Cathode"
- board text added: "ON-OFF"
- board text added: "VIN-GND-VOUT"
